Commit message: Add files via upload

File: urdf/robot3.urdf (robot description, URDF)
Before this commit: robot m2wr, 9 links, 8 joints
Links:
- added link arm_link_04, mass 0.005; collision box size=0.034 0.2 0.08; visual box size=0.034 0.2 0.08
- added link left_grip_link, mass 0.001; collision box size=0.001 0.001 0.001; visual box size=0.001 0.001 0.001
- added link right_grip_link, mass 0.001; collision box size=0.001 0.001 0.001; visual box size=0.001 0.001 0.001
- link arm_link_01: geometry collision cylinder length=0.25 radius=0.04; visual cylinder length=0.25 radius=0.04
- link arm_link_02: geometry collision cylinder length=0.25 radius=0.04; visual cylinder length=0.25 radius=0.04
- link arm_link_03: geometry collision cylinder length=0.25 radius=0.04; visual cylinder length=0.25 radius=0.04
- link camera_link: mass 0.025 -> 1e-5; geometry collision box size=0.05 0.05 0.05; visual box size=0.05 0.05 0.05
Joints:
- added joint arm_joint_04: type revolute, parent arm_link_03, child arm_link_04, origin xyz=0 0 0.25 rpy=0 0 0, axis 1 0 0, limit lower=-1.57 upper=1.57 effort=1000.0 velocity=0.5
- added joint left_grip_joint: type prismatic, parent arm_link_04, child left_grip_link, origin xyz=-0.015 0 0.0 rpy=0 0 0, axis 1 0 0, limit lower=-0.035 upper=0.04 effort=1000.0 velocity=6.5
- added joint right_grip_joint: type prismatic, parent arm_link_04, child right_grip_link, origin xyz=-0.015 0 0.0 rpy=0 0 0, axis 1 0 0, limit lower=-0.04 upper=0.035 effort=1000.0 velocity=6.5
- joint arm_joint_01: origin xyz=0 0 0.09 rpy=0 0 0 -> xyz=0 0 0.05 rpy=0 0 0
- joint arm_joint_02: origin xyz=0 0 0.04 rpy=0 0 0 -> xyz=0 0 0.25 rpy=0 0 0
- joint arm_joint_03: origin xyz=0 0 0.08 rpy=0 0 0 -> xyz=0 0 0.25 rpy=0 0 0
- joint camera_joint: axis 1 0 0 -> 0 1 0; origin xyz=0 0 0.08 rpy=0 0 0 -> xyz=0 0 0.0 rpy=0 0 0.05; parent arm_link_03 -> arm_link_04
