Commit message: works with moveit- no collision

File: urdf/myrobot3.xacro (robot description, xacro)
@@ -188,5 +188,5 @@
   	<axis xyz="1 0 0"/>
   	<limit effort="1000.0" lower="-1.8" upper="1.8" velocity="0.2"/>
-  	<origin rpy="0 0 0" xyz="0 0 0.25"/>
+  	<origin rpy="0 0 0" xyz="0 0 0.05"/>
   	<parent link="arm_link_01"/>
   	<child link="arm_link_02"/>

File: urdf/robot3.urdf (robot description, URDF)
Before this commit: robot myrobot3, 12 links, 11 joints
Links:
- link arm_link_04: geometry collision box size=0.0 0.0 0.0; visual box size=0.034 0.2 0.08
- link camera_link: geometry collision box size=0.0 0.0 0.0; visual box size=0.05 0.05 0.05

File: urdf/robot31.urdf (robot description, URDF)
Before this commit: robot myrobot3, 12 links, 11 joints
Links:
- link arm_link_01: geometry collision cylinder length=0.0 radius=0.0; visual cylinder length=0.25 radius=0.04
- link arm_link_02: geometry collision cylinder length=0.0 radius=0.0; visual cylinder length=0.25 radius=0.04
- link arm_link_03: geometry collision cylinder length=0.0 radius=0.0; visual cylinder length=0.25 radius=0.04
- link arm_link_04: geometry collision box size=0.0 0.0 0.0; visual box size=0.034 0.2 0.08
- link camera_link: geometry collision box size=0.0 0.0 0.0; visual box size=0.05 0.05 0.05
