Commit message: slam

File: urdf/robot31.urdf (robot description, URDF)
Before this commit: robot myrobot3, 12 links, 11 joints
Joints:
- joint joint_left_wheel: child link_left_wheel -> link_right_wheel; origin xyz=-0.05 -0.15 0 rpy=0 0 0 -> xyz=-0.05 0.15 0 rpy=0 0 0
- joint joint_right_wheel: child link_right_wheel -> link_left_wheel; origin xyz=-0.05 0.15 0 rpy=0 0 0 -> xyz=-0.05 -0.15 0 rpy=0 0 0
